File: eagle/stageboy-edcor-dips.sch (EAGLE design)
At the start: 39 parts, among them IC1 MEGA8-P, IC2 7805TV, J1 PWR, Q1 16MHz, X1 MIDI IN, X2 MIDI OUT, X4 22-23-2021, X6 GBIO

Commit message: Added 5VDC Header
Parts:
- added 5VDC: DCPWR, pinhead:PINHD-1X2
Connections:
- net +5V: now also 5VDC.1
- net GND: now also 5VDC.2
Changed lines of the file:
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@@
 <part name="R4" library="resistor" deviceset="R-US_" device="0204/7" value="220"/>
 <part name="R5" library="resistor" deviceset="R-US_" device="0204/7" value="220"/>
+<part name="5VDC" library="pinhead" deviceset="PINHD-1X2" device="" value="DCPWR"/>
+<part name="SUPPLY28" library="supply2" deviceset="+5V" device=""/>
+<part name="SUPPLY29" library="supply2" deviceset="GND" device=""/>
 </parts>
 <sheets>
@@
 <instance part="R4" gate="G$1" x="157.48" y="27.94" rot="R180"/>
 <instance part="R5" gate="G$1" x="147.32" y="25.4" rot="R180"/>
+<instance part="5VDC" gate="G$1" x="101.6" y="137.16"/>
+<instance part="SUPPLY28" gate="+5V" x="86.36" y="139.7" rot="R90"/>
+<instance part="SUPPLY29" gate="GND" x="76.2" y="137.16" rot="R270"/>
 </instances>
 <busses>
@@
 <pinref part="LED2" gate="G$1" pin="C"/>
 <pinref part="SUPPLY21" gate="GND" pin="GND"/>
+</segment>
+<segment>
+<pinref part="5VDC" gate="G$1" pin="2"/>
+<pinref part="SUPPLY29" gate="GND" pin="GND"/>
+<wire x1="99.06" y1="137.16" x2="78.74" y2="137.16" width="0.1524" layer="91"/>
 </segment>
 </net>
@@
 <junction x="233.68" y="35.56"/>
 </segment>
+<segment>
+<pinref part="5VDC" gate="G$1" pin="1"/>
+<pinref part="SUPPLY28" gate="+5V" pin="+5V"/>
+<wire x1="99.06" y1="139.7" x2="88.9" y2="139.7" width="0.1524" layer="91"/>
+</segment>
 </net>

Commit message: Added 5VDC Header
Parts:
- removed 5VDC: DCPWR, pinhead:PINHD-1X2
- added X3: DCPWR, con-molex:22-23-2021
- renumbered MIDIIN to MIDI-IN, MIDIOUT to MIDI-OUT
Connections:
- net +5V: now also X3-1.S; no longer 5VDC.1
- net GND: now also X3-2.S; no longer 5VDC.2
Changed lines of the file:
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@@
 <part name="SUPPLY20" library="supply2" deviceset="+5V" device=""/>
 <part name="SUPPLY22" library="supply2" deviceset="+5V" device=""/>
-<part name="MIDIOUT" library="pinhead" deviceset="PINHD-1X3" device="" value="MIDI OUT"/>
+<part name="MIDI-OUT" library="pinhead" deviceset="PINHD-1X3" device="" value="MIDI OUT"/>
 <part name="SUPPLY24" library="supply2" deviceset="+5V" device=""/>
 <part name="X2" library="con-hirschmann" deviceset="MAB5SH" device="" value="MIDI OUT"/>
-<part name="MIDIIN" library="pinhead" deviceset="PINHD-1X2" device="" value="MIDI IN"/>
+<part name="MIDI-IN" library="pinhead" deviceset="PINHD-1X2" device="" value="MIDI IN"/>
 <part name="C6" library="resistor" deviceset="CPOL-US" device="E2.5-6" value="22uF"/>
 <part name="SUPPLY16" library="supply2" deviceset="GND" device=""/>
@@
 <part name="R4" library="resistor" deviceset="R-US_" device="0204/7" value="220"/>
 <part name="R5" library="resistor" deviceset="R-US_" device="0204/7" value="220"/>
-<part name="5VDC" library="pinhead" deviceset="PINHD-1X2" device="" value="DCPWR"/>
 <part name="SUPPLY28" library="supply2" deviceset="+5V" device=""/>
 <part name="SUPPLY29" library="supply2" deviceset="GND" device=""/>
+<part name="X3" library="con-molex" deviceset="22-23-2021" device="" value="DCPWR"/>
 </parts>
 <sheets>
@@
 <instance part="SUPPLY20" gate="+5V" x="157.48" y="127"/>
 <instance part="SUPPLY22" gate="+5V" x="101.6" y="124.46" rot="R270"/>
-<instance part="MIDIOUT" gate="A" x="238.76" y="119.38"/>
+<instance part="MIDI-OUT" gate="A" x="238.76" y="119.38"/>
 <instance part="SUPPLY24" gate="+5V" x="223.52" y="99.06" rot="R270"/>
 <instance part="X2" gate="G$1" x="185.42" y="119.38" rot="R270"/>
-<instance part="MIDIIN" gate="G$1" x="304.8" y="71.12"/>
+<instance part="MIDI-IN" gate="G$1" x="304.8" y="71.12"/>
 <instance part="C6" gate="G$1" x="86.36" y="119.38"/>
 <instance part="SUPPLY16" gate="GND" x="86.36" y="111.76"/>
@@
 <instance part="R4" gate="G$1" x="157.48" y="27.94" rot="R180"/>
 <instance part="R5" gate="G$1" x="147.32" y="25.4" rot="R180"/>
-<instance part="5VDC" gate="G$1" x="101.6" y="137.16"/>
 <instance part="SUPPLY28" gate="+5V" x="86.36" y="139.7" rot="R90"/>
 <instance part="SUPPLY29" gate="GND" x="76.2" y="137.16" rot="R270"/>
+<instance part="X3" gate="-1" x="101.6" y="139.7"/>
+<instance part="X3" gate="-2" x="101.6" y="137.16"/>
 </instances>
 <busses>
@@
 </segment>
 <segment>
-<pinref part="5VDC" gate="G$1" pin="2"/>
 <pinref part="SUPPLY29" gate="GND" pin="GND"/>
 <wire x1="99.06" y1="137.16" x2="78.74" y2="137.16" width="0.1524" layer="91"/>
+<pinref part="X3" gate="-2" pin="S"/>
 </segment>
 </net>
@@
 </segment>
 <segment>
-<pinref part="5VDC" gate="G$1" pin="1"/>
 <pinref part="SUPPLY28" gate="+5V" pin="+5V"/>
 <wire x1="99.06" y1="139.7" x2="88.9" y2="139.7" width="0.1524" layer="91"/>
+<pinref part="X3" gate="-1" pin="S"/>
 </segment>
 </net>
@@
 <pinref part="D1" gate="G$1" pin="A"/>
 <pinref part="X1" gate="G$1" pin="5"/>
-<pinref part="MIDIIN" gate="G$1" pin="1"/>
+<pinref part="MIDI-IN" gate="G$1" pin="1"/>
 </segment>
 </net>
@@
 <junction x="276.86" y="53.34"/>
 <pinref part="R9" gate="G$1" pin="2"/>
-<pinref part="MIDIIN" gate="G$1" pin="2"/>
+<pinref part="MIDI-IN" gate="G$1" pin="2"/>
 <pinref part="X1" gate="G$1" pin="4"/>
 </segment>
@@
 <pinref part="IC1" gate="G$1" pin="PD1(TXD)"/>
 <pinref part="X2" gate="G$1" pin="5"/>
-<pinref part="MIDIOUT" gate="A" pin="1"/>
+<pinref part="MIDI-OUT" gate="A" pin="1"/>
 </segment>
 </net>
@@
 <wire x1="210.82" y1="99.06" x2="208.28" y2="99.06" width="0.1524" layer="91"/>
 <junction x="208.28" y="99.06"/>
-<pinref part="MIDIOUT" gate="A" pin="3"/>
+<pinref part="MIDI-OUT" gate="A" pin="3"/>
 <pinref part="X2" gate="G$1" pin="4"/>
 <pinref part="R10" gate="G$1" pin="2"/>
@@
 <net name="N$43" class="0">
 <segment>
-<pinref part="MIDIOUT" gate="A" pin="2"/>
+<pinref part="MIDI-OUT" gate="A" pin="2"/>
 <wire x1="236.22" y1="119.38" x2="203.2" y2="119.38" width="0.1524" layer="91"/>
 <wire x1="203.2" y1="119.38" x2="203.2" y2="101.6" width="0.1524" layer="91"/>

Commit message: Added side panels, minor layout changes to board
Parts:
- removed J1: PWR, con-jack:DCJ0303
- removed LED1: (no value), led:LED3MM
- removed R4: 220, resistor:R-US_0204/7
- added J2: DCJ0202, con-jack:DCJ0202
Connections:
- removed net N$5: LED1.A, R4.1
- net GND: no longer LED1.C
- net N$17: no longer R4.2
- net N$38: now also J2.3; no longer J1.3
- net N$39: now also J2.1; no longer J1.1
Changed lines of the file:
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@@
 <part name="SUPPLY6" library="supply2" deviceset="GND" device=""/>
 <part name="SUPPLY7" library="supply2" deviceset="GND" device=""/>
-<part name="J1" library="con-jack" deviceset="DCJ0303" device="" value="PWR"/>
 <part name="B1" library="rectifier" deviceset="RB1A" device="" value="B1"/>
 <part name="C7" library="resistor" deviceset="CPOL-US" device="E3.5-10" value="2200uF"/>
@@
 <part name="SUPPLY23" library="supply2" deviceset="GND" device=""/>
 <part name="SUPPLY25" library="supply2" deviceset="+5V" device=""/>
-<part name="LED1" library="led" deviceset="LED" device="3MM"/>
 <part name="LED2" library="led" deviceset="LED" device="3MM"/>
-<part name="SUPPLY14" library="supply2" deviceset="GND" device=""/>
 <part name="SUPPLY21" library="supply2" deviceset="GND" device=""/>
-<part name="R4" library="resistor" deviceset="R-US_" device="0204/7" value="220"/>
 <part name="R5" library="resistor" deviceset="R-US_" device="0204/7" value="220"/>
 <part name="SUPPLY28" library="supply2" deviceset="+5V" device=""/>
 <part name="SUPPLY29" library="supply2" deviceset="GND" device=""/>
 <part name="X3" library="con-molex" deviceset="22-23-2021" device="" value="DCPWR"/>
+<part name="J2" library="con-jack" deviceset="DCJ0202" device=""/>
 </parts>
 <sheets>
@@
 <instance part="SUPPLY6" gate="GND" x="73.66" y="111.76"/>
 <instance part="SUPPLY7" gate="GND" x="48.26" y="114.3"/>
-<instance part="J1" gate="G$1" x="-15.24" y="114.3" rot="MR180"/>
 <instance part="B1" gate="1" x="7.62" y="114.3" rot="R180"/>
 <instance part="C7" gate="G$1" x="22.86" y="119.38"/>
@@
 <instance part="SUPPLY23" gate="GND" x="205.74" y="10.16"/>
 <instance part="SUPPLY25" gate="+5V" x="241.3" y="35.56" rot="R270"/>
-<instance part="LED1" gate="G$1" x="165.1" y="20.32"/>
 <instance part="LED2" gate="G$1" x="154.94" y="20.32"/>
-<instance part="SUPPLY14" gate="GND" x="165.1" y="12.7"/>
 <instance part="SUPPLY21" gate="GND" x="154.94" y="12.7"/>
-<instance part="R4" gate="G$1" x="157.48" y="27.94" rot="R180"/>
 <instance part="R5" gate="G$1" x="147.32" y="25.4" rot="R180"/>
 <instance part="SUPPLY28" gate="+5V" x="86.36" y="139.7" rot="R90"/>
@@
 <instance part="X3" gate="-1" x="101.6" y="139.7"/>
 <instance part="X3" gate="-2" x="101.6" y="137.16"/>
+<instance part="J2" gate="G$1" x="-17.78" y="114.3"/>
 </instances>
 <busses>
@@
 <pinref part="R3" gate="G$1" pin="1"/>
 <pinref part="SUPPLY23" gate="GND" pin="GND"/>
-</segment>
-<segment>
-<pinref part="LED1" gate="G$1" pin="C"/>
-<pinref part="SUPPLY14" gate="GND" pin="GND"/>
 </segment>
 <segment>
@@
 <wire x1="134.62" y1="5.08" x2="139.7" y2="5.08" width="0.1524" layer="91"/>
 <wire x1="139.7" y1="5.08" x2="139.7" y2="27.94" width="0.1524" layer="91"/>
-<pinref part="R4" gate="G$1" pin="2"/>
-<wire x1="152.4" y1="27.94" x2="139.7" y2="27.94" width="0.1524" layer="91"/>
-<junction x="139.7" y="27.94"/>
 </segment>
 </net>
@@
 <wire x1="7.62" y1="119.38" x2="7.62" y2="121.92" width="0.1524" layer="91"/>
 <wire x1="7.62" y1="121.92" x2="-2.54" y2="121.92" width="0.1524" layer="91"/>
-<wire x1="-2.54" y1="121.92" x2="-2.54" y2="116.84" width="0.1524" layer="91"/>
-<pinref part="J1" gate="G$1" pin="3"/>
-<wire x1="-2.54" y1="116.84" x2="-7.62" y2="116.84" width="0.1524" layer="91"/>
+<wire x1="-2.54" y1="121.92" x2="-2.54" y2="114.3" width="0.1524" layer="91"/>
 <pinref part="X4" gate="-1" pin="S"/>
 <wire x1="-7.62" y1="121.92" x2="-2.54" y2="121.92" width="0.1524" layer="91"/>
 <junction x="-2.54" y="121.92"/>
+<wire x1="-2.54" y1="114.3" x2="-7.62" y2="114.3" width="0.1524" layer="91"/>
+<wire x1="-7.62" y1="114.3" x2="-7.62" y2="111.76" width="0.1524" layer="91"/>
+<pinref part="J2" gate="G$1" pin="3"/>
+<wire x1="-7.62" y1="111.76" x2="-10.16" y2="111.76" width="0.1524" layer="91"/>
 </segment>
 </net>
 <net name="N$39" class="0">
 <segment>
-<pinref part="J1" gate="G$1" pin="1"/>
-<wire x1="-7.62" y1="111.76" x2="-2.54" y2="111.76" width="0.1524" layer="91"/>
 <wire x1="-2.54" y1="111.76" x2="-2.54" y2="106.68" width="0.1524" layer="91"/>
 <pinref part="B1" gate="1" pin="AC1"/>
@@
 <wire x1="-7.62" y1="106.68" x2="-2.54" y2="106.68" width="0.1524" layer="91"/>
 <junction x="-2.54" y="106.68"/>
+<pinref part="J2" gate="G$1" pin="1"/>
+<wire x1="-10.16" y1="116.84" x2="-5.08" y2="116.84" width="0.1524" layer="91"/>
+<wire x1="-5.08" y1="116.84" x2="-5.08" y2="111.76" width="0.1524" layer="91"/>
+<wire x1="-5.08" y1="111.76" x2="-2.54" y2="111.76" width="0.1524" layer="91"/>
 </segment>
 </net>
@@
 </segment>
 </net>
-<net name="N$5" class="0">
-<segment>
-<pinref part="R4" gate="G$1" pin="1"/>
-<pinref part="LED1" gate="G$1" pin="A"/>
-<wire x1="162.56" y1="27.94" x2="165.1" y2="27.94" width="0.1524" layer="91"/>
-<wire x1="165.1" y1="27.94" x2="165.1" y2="22.86" width="0.1524" layer="91"/>
-</segment>
-</net>

Commit message: Added silkscreen and made minor formatting changes
Parts:
- R10: value R10 -> 220
- R8: value R8 -> 270
- R9: value R9 -> 220
- renumbered LED2 to LED, X3 to 5VDC
Changed lines of the file:
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@@
 <part name="OK1" library="optocoupler" deviceset="6N138" device=""/>
 <part name="SUPPLY8" library="supply2" deviceset="GND" device=""/>
-<part name="R8" library="resistor" deviceset="R-US_" device="0204/7" value="R8"/>
+<part name="R8" library="resistor" deviceset="R-US_" device="0204/7" value="270"/>
 <part name="D1" library="diode" deviceset="1N4148" device="DO35-7"/>
 <part name="X1" library="con-hirschmann" deviceset="MAB5SH" device="" value="MIDI IN"/>
-<part name="R9" library="resistor" deviceset="R-US_" device="0204/7" value="R9"/>
-<part name="R10" library="resistor" deviceset="R-US_" device="0204/7" value="R10"/>
+<part name="R9" library="resistor" deviceset="R-US_" device="0204/7" value="220"/>
+<part name="R10" library="resistor" deviceset="R-US_" device="0204/7" value="220"/>
 <part name="Q1" library="crystal" deviceset="CRYSTAL" device="HC49S" value="16MHz"/>
 <part name="SUPPLY17" library="supply2" deviceset="GND" device=""/>
@@
 <part name="SUPPLY23" library="supply2" deviceset="GND" device=""/>
 <part name="SUPPLY25" library="supply2" deviceset="+5V" device=""/>
-<part name="LED2" library="led" deviceset="LED" device="3MM"/>
+<part name="LED" library="led" deviceset="LED" device="3MM"/>
 <part name="SUPPLY21" library="supply2" deviceset="GND" device=""/>
 <part name="R5" library="resistor" deviceset="R-US_" device="0204/7" value="220"/>
 <part name="SUPPLY28" library="supply2" deviceset="+5V" device=""/>
 <part name="SUPPLY29" library="supply2" deviceset="GND" device=""/>
-<part name="X3" library="con-molex" deviceset="22-23-2021" device="" value="DCPWR"/>
+<part name="5VDC" library="con-molex" deviceset="22-23-2021" device="" value="DCPWR"/>
 <part name="J2" library="con-jack" deviceset="DCJ0202" device=""/>
 </parts>
@@
 <instance part="SUPPLY23" gate="GND" x="205.74" y="10.16"/>
 <instance part="SUPPLY25" gate="+5V" x="241.3" y="35.56" rot="R270"/>
-<instance part="LED2" gate="G$1" x="154.94" y="20.32"/>
+<instance part="LED" gate="G$1" x="154.94" y="20.32"/>
 <instance part="SUPPLY21" gate="GND" x="154.94" y="12.7"/>
 <instance part="R5" gate="G$1" x="147.32" y="25.4" rot="R180"/>
 <instance part="SUPPLY28" gate="+5V" x="86.36" y="139.7" rot="R90"/>
 <instance part="SUPPLY29" gate="GND" x="76.2" y="137.16" rot="R270"/>
-<instance part="X3" gate="-1" x="101.6" y="139.7"/>
-<instance part="X3" gate="-2" x="101.6" y="137.16"/>
+<instance part="5VDC" gate="-1" x="101.6" y="139.7"/>
+<instance part="5VDC" gate="-2" x="101.6" y="137.16"/>
 <instance part="J2" gate="G$1" x="-17.78" y="114.3"/>
 </instances>
@@
 </segment>
 <segment>
-<pinref part="LED2" gate="G$1" pin="C"/>
+<pinref part="LED" gate="G$1" pin="C"/>
 <pinref part="SUPPLY21" gate="GND" pin="GND"/>
 </segment>
@@
 <pinref part="SUPPLY29" gate="GND" pin="GND"/>
 <wire x1="99.06" y1="137.16" x2="78.74" y2="137.16" width="0.1524" layer="91"/>
-<pinref part="X3" gate="-2" pin="S"/>
+<pinref part="5VDC" gate="-2" pin="S"/>
 </segment>
 </net>
@@
 <pinref part="SUPPLY28" gate="+5V" pin="+5V"/>
 <wire x1="99.06" y1="139.7" x2="88.9" y2="139.7" width="0.1524" layer="91"/>
-<pinref part="X3" gate="-1" pin="S"/>
+<pinref part="5VDC" gate="-1" pin="S"/>
 </segment>
 </net>
@@
 <segment>
 <pinref part="R5" gate="G$1" pin="1"/>
-<pinref part="LED2" gate="G$1" pin="A"/>
+<pinref part="LED" gate="G$1" pin="A"/>
 <wire x1="152.4" y1="25.4" x2="154.94" y2="25.4" width="0.1524" layer="91"/>
 <wire x1="154.94" y1="25.4" x2="154.94" y2="22.86" width="0.1524" layer="91"/>
